Commit message: fix: Correct base link name from delto_base_link to l_dg_base

File: dg3f_b_driver/urdf/dg3f_b_mock.xacro (robot description, xacro)
@@ -7,5 +7,5 @@
     <joint name="base_joint" type="fixed">
         <parent link="base_link"/>
-        <child link="delto_base_link"/>
+        <child link="l_dg_base"/>
         <origin xyz="0 0 0" rpy="0 0 0"/>
     </joint>

File: dg3f_b_driver/urdf/dg3f_b_ros2_control.xacro (robot description, xacro)
@@ -14,5 +14,5 @@
     <joint name="base_joint" type="fixed">
         <parent link="base_link"/>
-        <child link="delto_base_link"/>
+        <child link="l_dg_base"/>
         <origin xyz="0 0 0" rpy="0 0 0"/>
     </joint>
